File: electronics/battery_management.kicad_sch (KiCad schematic)
At the start: 29 parts, among them IC3 CN3058E, IC4 HY2112, Q1 2N7002, Q4 FS8205, Q5 2N7002, SW2 SW_SPDT, U3 INA219AxD, U4 MT3608

Commit message: First draft of schematic and PCB of controller board
Parts:
- D2: footprint (none) -> Capacitor_SMD:C_0603_1608Metric_Pad1.08x0.95mm_HandSolder
- renumbered BAT2 to BAT1, C6 to C1, C8 to C2, C1 to C3, C7 to C4, C2 to C5, IC3 to IC1, IC4 to IC2, L2 to L1, Q4 to Q1, Q1 to Q2, Q5 to Q3, R19 to R10, R13 to R11, R21 to R12, R20 to R13, R16 to R2, R17 to R3, R2 to R4, R1 to R5, R18 to R6, R3 to R7, R6 to R8, R10 to R9, SW2 to SW1, U4 to U1, U3 to U2

Commit message: performed CRC check and fixed errors
Parts:
- D2: footprint Capacitor_SMD:C_0603_1608Metric_Pad1.08x0.95mm_HandSolder -> LED_SMD:LED_0603_1608Metric_Pad1.05x0.95mm_HandSolder
Changed lines of the file:
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@@
 			)
 		)
-		(property "Footprint" "Capacitor_SMD:C_0603_1608Metric_Pad1.08x0.95mm_HandSolder"
+		(property "Footprint" "LED_SMD:LED_0603_1608Metric_Pad1.05x0.95mm_HandSolder"
 			(at 147.32 55.88 0)
 			(effects

Commit message: started with v1.1 pcb fixes
Parts:
- added D4: SS34A, Chof747 Footprints:DIOM5026X262N, symbol Chof747 passive:SS34A
- added D5: CHG, LED_THT:LED_D3.0mm, symbol Device:LED
- added D6: RDY, LED_THT:LED_D3.0mm, symbol Device:LED
- added R29: 1k, Resistor_SMD:R_0603_1608Metric_Pad0.98x0.95mm_HandSolder, symbol Device:R
- D2: footprint LED_SMD:LED_0603_1608Metric_Pad1.05x0.95mm_HandSolder -> LED_THT:LED_D3.0mm
Connections:
- net CHG_IND: now also D5.1 (K)
- net RDY_IND: now also D6.1 (K)
- net VBUS: now also D4.2 (A), R29.1; no longer C1.1, IC1.4 (VIN)
- new net: D5.2 (A), D6.2 (A), R29.2
- new net VBUS_CHG: C1.1, D4.1 (K), IC1.4 (VIN)
