File: electronics/kitchen-clock.kicad_sch (KiCad schematic)
At the start: 8 parts, among them J1 USB_B_Micro

Commit message: First draft of schematic and PCB of controller board
Parts:
- removed H1, H2, H3, H4: MountingHole, Chof747 Footprints:MountingHole_3.2mm_M3-smallBorder, symbol Mechanical:MountingHole
- renumbered D5 to D3
Other:
- sheet Microcontroller & Controls ports: added REN_BTN_IO10, REN_CLK_IO12; removed REN_BTN_IO12, REN_CLK_IO10

Commit message: started with v1.1 pcb fixes
Parts:
- D3: footprint LED_SMD:LED_0603_1608Metric_Pad1.05x0.95mm_HandSolder -> LED_THT:LED_D3.0mm
Changed lines of the file:
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@@
 			)
 		)
-		(property "Footprint" "LED_SMD:LED_0603_1608Metric_Pad1.05x0.95mm_HandSolder"
+		(property "Footprint" "LED_THT:LED_D3.0mm"
 			(at 50.8 173.99 0)
 			(effects
