File: electronics/mcu.kicad_sch (KiCad schematic)
At the start: 6 parts, among them IC1 ESP32-S3-WROOM-1-N8R8, J8 CONN_PGR, SW1 Reset

Commit message: First draft of schematic and PCB of controller board
Parts:
- added C10, C11: 20p, Capacitor_SMD:C_0603_1608Metric_Pad1.08x0.95mm_HandSolder, symbol Device:C
- added C8, C9: 1uF, Capacitor_SMD:C_0603_1608Metric_Pad1.08x0.95mm_HandSolder, symbol Device:C
- added IC4: ME6211C33M5G-N, SOT95P270X145-5N, symbol Chof747 Voltage Regulators:ME6211C33M5G-N
- added R25, R26: 10k, Resistor_SMD:R_0603_1608Metric_Pad0.98x0.95mm_HandSolder, symbol Device:R
- added R27, R28: 22, Resistor_SMD:R_0603_1608Metric_Pad0.98x0.95mm_HandSolder, symbol Device:R
- added U3: USBLC6-2SC6, Package_TO_SOT_SMD:SOT-23-6, symbol Power_Protection:USBLC6-2SC6
- C6: renamed from C4; footprint (none) -> Capacitor_SMD:C_0603_1608Metric_Pad1.08x0.95mm_HandSolder
- C7: renamed from C3; footprint (none) -> Capacitor_SMD:C_0603_1608Metric_Pad1.08x0.95mm_HandSolder
- J8: footprint (none) -> Connector_PinSocket_2.54mm:PinSocket_1x04_P2.54mm_Vertical
- R1: renamed from R4; footprint (none) -> Resistor_SMD:R_0603_1608Metric_Pad0.98x0.95mm_HandSolder
- SW2: renamed from SW1; footprint (none) -> Chof747 Footprints:1TS003B-2500-3500A-CT (SMD Right Angle Tactile Switch)
- renumbered IC1 to IC3
Connections:
- net +3V3: now also C9.1, IC4.5 (VOUT), R25.1, R26.1
- net GND: now also C10.2, C11.2, C8.2, C9.2, IC4.2 (VSS), U3.2 (GND)
- net SCL: now also R26.2
- net SDA: now also R25.2
- net USB_N: now also U3.1 (I/O1); no longer IC3.13 (IO19)
- net USB_P: now also U3.3 (I/O2); no longer IC3.14 (IO20)
- net REN_BTN_IO12 renamed REN_CLK_IO12
- net REN_CLK_IO10 renamed REN_BTN_IO10
- new net +5V: C8.1, IC4.1 (VIN), IC4.3 (CE)
- new net USBPROT_N: C10.1, R27.1, U3.6 (I/O1)
- new net USBPROT_P: C11.1, R28.1, U3.4 (I/O2)
- new net USB_PROT_N: IC3.13 (IO19), R27.2
- new net USB_PROT_P: IC3.14 (IO20), R28.2
- new net VBUS: U3.5 (VBUS)
Other:
- moved on the sheet: C6, C7, IC3, J8, R1, SW2

Commit message: started with v1.1 pcb fixes
Connections:
- net ~{RESET}: now reaches C6.1, IC3.3 (EN), R1.2, SW2.2
Changed lines of the file:
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@@
+	(wire
+		(pts
+			(xy 26.67 43.18) (xy 31.75 43.18)
+		)
+		(stroke
+			(width 0)
+			(type default)
+		)
+	)
 	(wire
 		(pts
@@
 			(effects
 				(font
+					(size 1.27 1.27)
+				)
+				(justify right)
+				(hide yes)
+			)
+		)
+	)
+	(global_label "~{RESET}"
+		(shape input)
+		(at 26.67 43.18 180)
+		(effects
+			(font
+				(size 1.27 1.27)
+			)
+			(justify right)
+		)
+		(property "Intersheetrefs" "${INTERSHEET_REFS}"
+			(at 43.4002 86.36 0)
+			(effects
+				(font
