File: electronics/peripherals.kicad_sch (KiCad schematic)
At the start: 23 parts, among them J2 Temp 1, J3 Temp 2, J4 CONN_MOD, J5 CONN_ENC, J6 CONN_DISPL, J7 CONN_SERVO, Q2 SS8050-G, Q3 SS8050-G, Q6 AO3401A, Q7 SS8050-G, Q8 AO3401A, U1 ADS1115IDGS

Commit message: First draft of schematic and PCB of controller board
Parts:
- J4: footprint (none) -> Connector_PinSocket_2.54mm:PinSocket_1x02_P2.54mm_Vertical
- J5: footprint (none) -> Connector_PinSocket_2.54mm:PinSocket_1x05_P2.54mm_Vertical
- J6: footprint (none) -> Connector_PinSocket_2.54mm:PinSocket_1x08_P2.54mm_Vertical
- J7: footprint (none) -> Connector_PinSocket_2.54mm:PinSocket_1x03_P2.54mm_Vertical
- renumbered Q3 to Q4, Q7 to Q5, Q2 to Q6, Q6 to Q7, R5 to R16, R7 to R17, R11 to R18, R12 to R19, R8 to R20, R9 to R21, U1 to U4
Connections:
- net PWM_SERVO: now also J7.2 (Pin_2); no longer J7.1 (Pin_1)
- net SERVO_VCC: now also J7.1 (Pin_1); no longer J7.2 (Pin_2)
- net TEMP1: now also U4.7 (AIN3); no longer U4.5 (AIN1)
Changed lines of the file:
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@@
 	)
 	(no_connect
-		(at 81.28 172.72)
+		(at 81.28 167.64)
 	)
 	(wire
@@
 	(wire
 		(pts
-			(xy 81.28 167.64) (xy 69.85 167.64)
-		)
-		(stroke
-			(width 0)
-			(type default)
-		)
-	)
-	(wire
-		(pts
 			(xy 81.28 88.9) (xy 74.93 88.9)
 		)
@@
 	(wire
 		(pts
-			(xy 48.26 156.21) (xy 48.26 160.02)
+			(xy 250.19 147.32) (xy 252.73 147.32)
 		)
 		(stroke
@@
 	(wire
 		(pts
-			(xy 176.53 91.44) (xy 173.99 91.44)
+			(xy 48.26 156.21) (xy 48.26 160.02)
 		)
 		(stroke
@@
 	(wire
 		(pts
-			(xy 176.53 78.74) (xy 176.53 91.44)
+			(xy 176.53 77.47) (xy 176.53 88.9)
 		)
 		(stroke
@@
 	(wire
 		(pts
-			(xy 250.19 147.32) (xy 252.73 147.32)
-		)
-		(stroke
-			(width 0)
-			(type default)
-		)
-	)
-	(wire
-		(pts
 			(xy 252.73 26.67) (xy 252.73 34.29)
 		)
@@
 	(wire
 		(pts
-			(xy 57.15 176.53) (xy 69.85 176.53)
+			(xy 57.15 176.53) (xy 81.28 176.53)
 		)
 		(stroke
@@
 	(wire
 		(pts
-			(xy 69.85 167.64) (xy 69.85 176.53)
-		)
-		(stroke
-			(width 0)
-			(type default)
-		)
-	)
-	(wire
-		(pts
 			(xy 43.18 91.44) (xy 39.37 91.44)
 		)
@@
 	(wire
 		(pts
-			(xy 173.99 88.9) (xy 180.34 88.9)
+			(xy 119.38 106.68) (xy 129.54 106.68)
 		)
 		(stroke
@@
 	(wire
 		(pts
-			(xy 119.38 106.68) (xy 129.54 106.68)
+			(xy 123.19 78.74) (xy 123.19 91.44)
 		)
 		(stroke
@@
 	(wire
 		(pts
-			(xy 123.19 78.74) (xy 123.19 91.44)
+			(xy 119.38 96.52) (xy 132.08 96.52)
 		)
 		(stroke
@@
 	(wire
 		(pts
-			(xy 119.38 96.52) (xy 132.08 96.52)
+			(xy 123.19 91.44) (xy 119.38 91.44)
 		)
 		(stroke
@@
 	(wire
 		(pts
-			(xy 123.19 91.44) (xy 119.38 91.44)
+			(xy 173.99 88.9) (xy 176.53 88.9)
 		)
 		(stroke
@@
 	(wire
 		(pts
+			(xy 173.99 91.44) (xy 180.34 91.44)
+		)
+		(stroke
+			(width 0)
+			(type default)
+		)
+	)
+	(wire
+		(pts
 			(xy 260.35 97.79) (xy 264.16 97.79)
 		)
@@
 	(wire
 		(pts
+			(xy 81.28 172.72) (xy 81.28 176.53)
+		)
+		(stroke
+			(width 0)
+			(type default)
+		)
+	)
+	(wire
+		(pts
 			(xy 101.6 170.18) (xy 106.68 170.18)
 		)
@@
 	)
 	(label "SERVO_VCC"
-		(at 176.53 78.74 0)
+		(at 176.53 77.47 0)
 		(fields_autoplaced yes)
 		(effects
@@
 	(hierarchical_label "PWM_SERVO"
 		(shape input)
-		(at 180.34 88.9 0)
+		(at 180.34 91.44 0)
 		(fields_autoplaced yes)
 		(effects
@@
 			)
 		)
-		(property "Footprint" ""
+		(property "Footprint" "Connector_PinSocket_2.54mm:PinSocket_1x05_P2.54mm_Vertical"
 			(at 69.85 93.98 0)
 			(effects
@@
 		(dnp no)
 		(fields_autoplaced yes)
-		(property "Reference" "R7"
+		(property "Reference" "R17"
 			(at 54.61 35.5599 0)
 			(effects
@@
 			(project "kitchen-clock"
 				(path "/e8426e51-e5a9-4642-8277-6d3f50e0e523/29f485c1-716a-4531-b037-6348eb8cbfa2"
-					(reference "R7")
+					(reference "R17")
 					(unit 1)
 				)
@@
 			)
 		)
-		(property "Footprint" ""
+		(property "Footprint" "Connector_PinSocket_2.54mm:PinSocket_1x03_P2.54mm_Vertical"
 			(at 168.91 91.44 0)
 			(effects
@@
 		(dnp no)
 		(fields_autoplaced yes)
-		(property "Reference" "Q2"
+		(property "Reference" "Q6"
 			(at 262.89 146.0499 0)
 			(effects
@@
 			(project "kitchen-clock"
 				(path "/e8426e51-e5a9-4642-8277-6d3f50e0e523/29f485c1-716a-4531-b037-6348eb8cbfa2"
-					(reference "Q2")
+					(reference "Q6")
 					(unit 1)
 				)
@@
 		(dnp no)
 		(fields_autoplaced yes)
-		(property "Reference" "R11"
+		(property "Reference" "R18"
 			(at 229.87 41.91 90)
 			(effects
@@
 			(project "kitchen-clock"
 				(path "/e8426e51-e5a9-4642-8277-6d3f50e0e523/29f485c1-716a-4531-b037-6348eb8cbfa2"
-					(reference "R11")
+					(reference "R18")
 					(unit 1)
 				)
@@
 		(dnp no)
 		(fields_autoplaced yes)
-		(property "Reference" "Q7"
+		(property "Reference" "Q5"
 			(at 245.11 97.7899 0)
 			(effects
@@
 			(project "kitchen-clock"
 				(path "/e8426e51-e5a9-4642-8277-6d3f50e0e523/29f485c1-716a-4531-b037-6348eb8cbfa2"
-					(reference "Q7")
+					(reference "Q5")
 					(unit 1)
 				)
@@
 		(dnp no)
 		(fields_autoplaced yes)
-		(property "Reference" "R9"
+		(property "Reference" "R21"
 			(at 257.81 130.8099 0)
 			(effects
@@
 			(project "kitchen-clock"
 				(path "/e8426e51-e5a9-4642-8277-6d3f50e0e523/29f485c1-716a-4531-b037-6348eb8cbfa2"
-					(reference "R9")
+					(reference "R21")
 					(unit 1)
 				)
@@
 			)
 		)
-		(property "Footprint" ""
+		(property "Footprint" "Connector_PinSocket_2.54mm:PinSocket_1x08_P2.54mm_Vertical"
 			(at 114.3 96.52 0)
 			(effects
@@
 		(on_board yes)
 		(dnp no)
-		(property "Reference" "Q6"
+		(property "Reference" "Q7"
 			(at 256.54 40.005 0)
 			(effects
@@
 			(project "kitchen-clock"
 				(path "/e8426e51-e5a9-4642-8277-6d3f50e0e523/29f485c1-716a-4531-b037-6348eb8cbfa2"
-					(reference "Q6")
+					(reference "Q7")
 					(unit 1)
 				)
@@
 		(dnp no)
 		(fields_autoplaced yes)
-		(property "Reference" "R8"
+		(property "Reference" "R20"
 			(at 246.38 140.97 90)
 			(effects
@@
 			(project "kitchen-clock"
 				(path "/e8426e51-e5a9-4642-8277-6d3f50e0e523/29f485c1-716a-4531-b037-6348eb8cbfa2"
-					(reference "R8")
+					(reference "R20")
 					(unit 1)
 				)
@@
 		(dnp no)
 		(fields_autoplaced yes)
-		(property "Reference" "U1"
+		(property "Reference" "U4"
 			(at 93.6341 152.4 0)
 			(effects
@@
 			(project ""
 				(path "/e8426e51-e5a9-4642-8277-6d3f50e0e523/29f485c1-716a-4531-b037-6348eb8cbfa2"
-					(reference "U1")
+					(reference "U4")
 					(unit 1)
 				)
@@
 		(dnp no)
 		(fields_autoplaced yes)
-		(property "Reference" "R12"
-			(at 243.84 31.115 0)
+		(property "Reference" "R19"
+			(at 243.84 30.4799 0)
 			(effects
 				(font
@@
 		)
 		(property "Value" "10k"
-			(at 243.84 33.655 0)
+			(at 243.84 33.0199 0)
 			(effects
 				(font
@@
 			(project "kitchen-clock"
 				(path "/e8426e51-e5a9-4642-8277-6d3f50e0e523/29f485c1-716a-4531-b037-6348eb8cbfa2"
-					(reference "R12")
+					(reference "R19")
 					(unit 1)
 				)
@@
 			)
 		)
-		(property "Footprint" ""
+		(property "Footprint" "Connector_PinSocket_2.54mm:PinSocket_1x02_P2.54mm_Vertical"
 			(at 34.29 91.44 0)
 			(effects
@@
 		(on_board yes)
 		(dnp no)
-		(property "Reference" "R5"
+		(property "Reference" "R16"
 			(at 46.99 38.1 90)
 			(effects
@@
 			(project "kitchen-clock"
 				(path "/e8426e51-e5a9-4642-8277-6d3f50e0e523/29f485c1-716a-4531-b037-6348eb8cbfa2"
-					(reference "R5")
+					(reference "R16")
 					(unit 1)
 				)
@@
 		(dnp no)
 		(fields_autoplaced yes)
-		(property "Reference" "Q3"
+		(property "Reference" "Q4"
 			(at 243.84 46.9899 0)
 			(effects
@@
 			(project "kitchen-clock"
 				(path "/e8426e51-e5a9-4642-8277-6d3f50e0e523/29f485c1-716a-4531-b037-6348eb8cbfa2"
-					(reference "Q3")
+					(reference "Q4")
 					(unit 1)
 				)

Commit message: Performed CRC and DRC on board + corrections
Parts:
- added C12: 0.1uF, Capacitor_SMD:C_0603_1608Metric_Pad1.08x0.95mm_HandSolder, symbol Device:C
Connections:
- net +3V3: now also C12.1
- net GND: now also C12.2
Changed lines of the file:
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@@
 	)
 	(junction
+		(at 91.44 148.59)
+		(diameter 0)
+		(color 0 0 0 0)
+	)
+	(junction
 		(at 241.3 39.37)
 		(diameter 0)
@@
 	(wire
 		(pts
-			(xy 91.44 146.05) (xy 91.44 154.94)
+			(xy 91.44 146.05) (xy 91.44 148.59)
 		)
 		(stroke
@@
 	(wire
 		(pts
+			(xy 91.44 148.59) (xy 111.76 148.59)
+		)
+		(stroke
+			(width 0)
+			(type default)
+		)
+	)
+	(wire
+		(pts
 			(xy 119.38 88.9) (xy 124.46 88.9)
 		)
@@
 	(wire
 		(pts
+			(xy 91.44 148.59) (xy 91.44 154.94)
+		)
+		(stroke
+			(width 0)
+			(type default)
+		)
+	)
+	(wire
+		(pts
 			(xy 173.99 91.44) (xy 180.34 91.44)
 		)
@@
 	)
 	(symbol
+		(lib_id "power:GND")
+		(at 111.76 156.21 0)
+		(unit 1)
+		(exclude_from_sim no)
+		(in_bom yes)
+		(on_board yes)
+		(dnp no)
+		(fields_autoplaced yes)
+		(property "Reference" "#PWR041"
+			(at 111.76 162.56 0)
+			(effects
+				(font
+					(size 1.27 1.27)
+				)
+				(hide yes)
+			)
+		)
+		(property "Value" "GND"
+			(at 111.76 161.29 0)
+			(effects
+				(font
+					(size 1.27 1.27)
+				)
+			)
+		)
+		(property "Footprint" ""
+			(at 111.76 156.21 0)
+			(effects
+				(font
+					(size 1.27 1.27)
+				)
+				(hide yes)
+			)
+		)
+		(property "Datasheet" ""
+			(at 111.76 156.21 0)
+			(effects
+				(font
+					(size 1.27 1.27)
+				)
+				(hide yes)
+			)
+		)
+		(property "Description" "Power symbol creates a global label with name \"GND\" , ground"
+			(at 111.76 156.21 0)
+			(effects
+				(font
+					(size 1.27 1.27)
+				)
+				(hide yes)
+			)
+		)
+		(pin "1"
+		)
+		(instances
+			(project ""
+				(path "/e8426e51-e5a9-4642-8277-6d3f50e0e523/29f485c1-716a-4531-b037-6348eb8cbfa2"
+					(reference "#PWR041")
+					(unit 1)
+				)
+			)
+		)
+	)
+	(symbol
 		(lib_id "Device:R")
 		(at 229.87 48.26 270)
@@
 					(unit 1)
 				)
+			)
+		)
+	)
+	(symbol
+		(lib_id "Device:C")
+		(at 111.76 152.4 0)
+		(unit 1)
+		(exclude_from_sim no)
+		(in_bom yes)
+		(on_board yes)
+		(dnp no)
+		(fields_autoplaced yes)
+		(property "Reference" "C12"
+			(at 115.57 151.1299 0)
+			(effects
+				(font
+					(size 1.27 1.27)
+				)
+				(justify left)
+			)
+		)
+		(property "Value" "0.1uF"
+			(at 115.57 153.6699 0)
+			(effects
+				(font
+					(size 1.27 1.27)
+				)
+				(justify left)
+			)
+		)
+		(property "Footprint" "Capacitor_SMD:C_0603_1608Metric_Pad1.08x0.95mm_HandSolder"
+			(at 112.7252 156.21 0)
+			(effects
+				(font
+					(size 1.27 1.27)
+				)
+				(hide yes)
+			)
+		)
+		(property "Datasheet" "~"
+			(at 111.76 152.4 0)
+			(effects
+				(font
+					(size 1.27 1.27)
+				)
+				(hide yes)
+			)
+		)
+		(property "Description" "Unpolarized capacitor"
+			(at 111.76 152.4 0)
+			(effects
+				(font
+					(size 1.27 1.27)
+				)
+				(hide yes)
+			)
+		)
+		(pin "1"
+		)
+		(pin "2"
+		)
+		(instances
+			(project ""
+				(path "/e8426e51-e5a9-4642-8277-6d3f50e0e523/29f485c1-716a-4531-b037-6348eb8cbfa2"
+					(reference "C12")
+					(unit 1)
+				)

Commit message: started with v1.1 pcb fixes
Parts:
- added J9: I2C, Connector_PinHeader_2.54mm:PinHeader_1x06_P2.54mm_Vertical, symbol Connector:Conn_01x06_Pin
- J4: value CONN_MOD -> MOD
- J5: value CONN_ENC -> ENC
- J6: value CONN_DISPL -> DISPL
- J7: value CONN_SERVO -> SERVO
Connections:
- net +3V3: now also J9.2 (Pin_2)
- net +5V: now also J9.6 (Pin_6)
- net GND: now also J9.1 (Pin_1)
- net SCL: now also J9.3 (Pin_3)
- net SDA: now also J9.4 (Pin_4)
- new net ~{RESET}: J9.5 (Pin_5)
