File: electronics/kitchen-clock.kicad_pcb (KiCad board)
At the start: 2 copper layers, 66.9 x 110 mm, 74 parts, among them IC1 CN3058E, IC2 HY2112, IC3 ESP32-S3-WROOM-1-N8R8, IC4 ME6211C33M5G-N, J1 USB_B_Micro, J2 Temp 1, J3 Temp 2, J4 CONN_MOD, J5 CONN_ENC, J6 CONN_DISPL, J7 CONN_SERVO, J8 CONN_PGR, Q1 FS8205, Q2 2N7002, Q3 2N7002, Q4 SS8050-G, Q5 SS8050-G, Q6 SS8050-G, Q7 AO3401A, Q8 AO3401A, SW1 SW_SPDT, SW2 Reset, U1 MT3608, U2 INA219AxD, U3 USBLC6-2SC6, U4 ADS1115IDGS

Commit message: started with v1.1 pcb fixes
Parts:
- added D4: SS34A, Chof747 Footprints:DIOM5026X262N, F.Cu at (188.2, 133.5)
- added D5: CHG, LED_THT:LED_D3.0mm, F.Cu at (190.8, 97.4)
- added D6: RDY, LED_THT:LED_D3.0mm, F.Cu at (190.8, 103.9)
- added J9: I2C, Connector_PinHeader_2.54mm:PinHeader_1x06_P2.54mm_Vertical, F.Cu at (187.4, 57.5)
- added R29: 1k, Resistor_SMD:R_0603_1608Metric_Pad0.98x0.95mm_HandSolder, F.Cu at (187.2, 101.8)
- D2, D3: footprint LED_SMD:LED_0603_1608Metric_Pad1.05x0.95mm_HandSolder -> LED_THT:LED_D3.0mm
- J4: value CONN_MOD -> MOD
- J5: value CONN_ENC -> ENC
- J6: value CONN_DISPL -> DISPL
- J7: value CONN_SERVO -> SERVO
- moved D2 56.4 mm to (190.8, 90.9)
- moved R6 56.0 mm to (187.2, 92.3)
- moved D3 21.0 mm to (190.8, 110.4), turned to -90 degrees
- moved R14 16.7 mm to (187.5, 112.7), turned to -90 degrees
Connections:
- net Net-(IC3-EN) renamed ~{RESET}
- C1 pad 1: VBUS -> /Battery Management/VBUS_CHG
- IC1 pad 4: VBUS -> /Battery Management/VBUS_CHG
Routing:
- net /Battery Management/VBAT: track 81.5 -> 140.2 mm, vias 0 -> 4
- net /Battery Management/CHG_IND: track 21.2 -> 70.9 mm, vias 4 -> 8
- net /Battery Management/RDY_IND: track 16.2 -> 58.0 mm, vias 2 -> 4
- net SCL: track 88.7 -> 112.6 mm, vias 2 -> 5
- net SDA: track 92.2 -> 113.6 mm, vias 2 -> 4
- net VBUS: track 54.0 -> 67.1 mm
- net Net-(D5-A): track 0.00 -> 11.3 mm
- net GND: track 43.0 -> 39.9 mm, vias 31 -> 29
- net +3V3: track 225.3 -> 228.1 mm
- net Net-(D2-A): track 1.86 -> 3.78 mm
- net Net-(D3-A): track 1.77 -> 3.61 mm
- net Net-(IC3-IO0): track 46.3 -> 48.1 mm
- net Net-(IC3-TXD0): track 35.6 -> 35.0 mm
- added copper zone on F.Cu, net /Battery Management/VBUS_CHG
Other:
- board text added: "3V3"
- board text added: "5V"
- board text added: "BTN"
- board text added: "CLK"
- board text added: "CS"
- board text added: "DAT"
- board text added: "G"
- board text added: "I0"
- board text added: "PWM"
- board text added: "PWR"
- board text added: "RS"
- board text added: "RST"
- board text added: "RX<"
- board text added: "SCL"
- board text added: "SDA"
- board text added: "TX>"
- board text removed: "+5V"
- board text removed: "GND"

Commit message: update on pcb design
Routing:
- net +5V: track 90.6 -> 126.8 mm, vias 4 -> 6
- net ~{RESET}: track 49.4 -> 83.8 mm, vias 4 -> 9
- net SDA: track 113.6 -> 140.3 mm, vias 4 -> 5
- net Net-(IC3-IO0): track 48.1 -> 47.4 mm
- net /Battery Management/VBAT: vias 4 -> 6
- net /Microcontroller & Controls/PWM_SERVO_IO47: vias 0 -> 2
